File: PCB_NeoPixel_Booster/PCB_NeoPixel_Booster.kicad_sch (KiCad schematic)
At the start: 17 parts, among them J1 Power_Input_Screw, J10 5V_Breakout, J11 Power_Input_Screw, J2 Power_Input_Barrel_Jack, J3 Vcc_Breakout, J4 LED_Strip_Connector, J5 Power_Input_Screw, J6 LED_Strip_Connector, J7 Data_Input, J8 5V_Breakout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

Commit message: Fix
Parts:
- removed J9: 5V_Breakout, Connector_PinHeader_2.54mm:PinHeader_1x02_P2.54mm_Vertical, symbol Connector:Conn_01x02_Pin
- removed JP1: Power_Selection, Jumper:SolderJumper-3_P2.0mm_Open_TrianglePad1.0x1.5mm, symbol Jumper:SolderJumper_3_Open
- added J12: REG_CONTROL, Connector_PinHeader_2.54mm:PinHeader_1x03_P2.54mm_Vertical, symbol Connector:Conn_01x03_Pin
- added R2, R4, R5, R6: 1k, Resistor_SMD:R_1206_3216Metric_Pad1.30x1.75mm_HandSolder, symbol Device:R
- added R3: 500, Resistor_SMD:R_1206_3216Metric_Pad1.30x1.75mm_HandSolder, symbol Device:R
- added U1: AP2210K-5.0, Package_TO_SOT_SMD:SOT-23-5, symbol Regulator_Linear:AP2204K-5.0
- J10, J8: value 5V_Breakout -> Power_Breakout
Connections:
- net +5V: now also J12.2 (Pin_2), U1.5 (VOUT); no longer J10.1 (Pin_1), J8.1 (Pin_1)
- net GND: now also J12.3 (Pin_3), U1.2 (GND)
- net LED_Input_ch1: now also J7.2 (Pin_2), U3.3 (2A); no longer J7.1 (Pin_1), U3.1 (1A)
- net LED_Input_ch2: now also J7.1 (Pin_1), U3.1 (1A); no longer J7.2 (Pin_2), U3.3 (2A)
- net LED_Output_ch1: now also U3.4 (2Y), R2.1, R4.1; no longer J4.2 (Pin_2), U3.6 (1Y)
- net LED_Output_ch2: now also U3.6 (1Y), R5.1, R6.1; no longer J6.2 (Pin_2), U3.4 (2Y)
- net VCC: now also J10.1 (Pin_1), J4.1 (Pin_1), J6.1 (Pin_1), J8.1 (Pin_1), R3.2, U1.1 (VIN)
- new net: J6.2 (Pin_2), R2.2, R4.2
- new net: J4.2 (Pin_2), R5.2, R6.2
- new net EN: J12.1 (Pin_1), R3.1, U1.3 (EN)
Other:
- note added: "C500758"
- moved on the sheet: J4, J6, J7, U3

Commit message: Fin
Other:
- moved on the sheet: J10, J11, J12, J4, J6, J7, J8, R2, R3, R4, R5, R6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

Commit message: Add Prod files
Parts:
- removed R3: 500, Resistor_SMD:R_1206_3216Metric_Pad1.30x1.75mm_HandSolder, symbol Device:R
- added R1: 1k, Resistor_SMD:R_1206_3216Metric_Pad1.30x1.75mm_HandSolder, symbol Device:R
- H1, H2, H4, H5, J1, J10, J11, J12, J2, J3, J4, J5, J6, J7, J8: now not fitted
- R2, R4, R5, R6: MPN (none) -> C4410
- U1: MPN (none) -> C500758
- U3: MPN (none) -> C347589
Connections:
- net EN: now also R1.1
- net VCC: now also R1.2
