File: PCB_NeoPixel_Booster/PCB_NeoPixel_Booster.kicad_pcb (KiCad board)
At the start: 2 copper layers, 49 x 56 mm, 17 parts, among them J1 Power_Input_Screw, J10 5V_Breakout, J11 Power_Input_Screw, J2 Power_Input_Barrel_Jack, J3 Vcc_Breakout, J4 LED_Strip_Connector, J5 Power_Input_Screw, J6 LED_Strip_Connector, J7 Data_Input, J8 5V_Breakout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

Commit message: Fix
Parts:
- removed J9: 5V_Breakout, Connector_PinHeader_2.54mm:PinHeader_1x02_P2.54mm_Vertical
- removed JP1: Power_Selection, Jumper:SolderJumper-3_P2.0mm_Open_TrianglePad1.0x1.5mm
- added H1: MountingHole, MountingHole:MountingHole_4.3mm_M4, F.Cu at (233.8, 54.5)
- added H1: MountingHole, MountingHole:MountingHole_4.3mm_M4, F.Cu at (300.5, 45.0)
- added H2: MountingHole, MountingHole:MountingHole_4.3mm_M4, F.Cu at (262.0, 91.0)
- added H2: MountingHole, MountingHole:MountingHole_4.3mm_M4, F.Cu at (195.3, 100.5)
- added H4: MountingHole, MountingHole:MountingHole_4.3mm_M4, F.Cu at (262.0, 45.0)
- added H4: MountingHole, MountingHole:MountingHole_4.3mm_M4, F.Cu at (195.3, 54.5)
- added H5: MountingHole, MountingHole:MountingHole_4.3mm_M4, F.Cu at (300.5, 91.0)
- added H5: MountingHole, MountingHole:MountingHole_4.3mm_M4, F.Cu at (233.8, 100.5)
- added J12: REG_CONTROL, Connector_PinHeader_2.54mm:PinHeader_1x03_P2.54mm_Vertical, F.Cu at (77.3, 79.0)
- added R2: 1k, Resistor_SMD:R_1206_3216Metric_Pad1.30x1.75mm_HandSolder, F.Cu at (64.8, 90.0)
- added R3: 500, Resistor_SMD:R_1206_3216Metric_Pad1.30x1.75mm_HandSolder, F.Cu at (74.0, 80.5)
- added R4: 1k, Resistor_SMD:R_1206_3216Metric_Pad1.30x1.75mm_HandSolder, F.Cu at (62.2, 90.0)
- added R5: 1k, Resistor_SMD:R_1206_3216Metric_Pad1.30x1.75mm_HandSolder, F.Cu at (68.5, 86.8)
- added R6: 1k, Resistor_SMD:R_1206_3216Metric_Pad1.30x1.75mm_HandSolder, F.Cu at (71.0, 86.8)
- added U1: AP2210K-5.0, Package_TO_SOT_SMD:SOT-23-5, F.Cu at (67.4, 80.3)
- J10, J8: value 5V_Breakout -> Power_Breakout
- moved J10 19.6 mm to (94.5, 89.6)
- moved J8 19.2 mm to (56.4, 79.5), turned to 0 degrees
- moved U3 5.86 mm to (63.0, 85.5)
- moved J7 4.02 mm to (56.4, 89.6)
Connections:
- J10 pad 1: +5V -> VCC
- J4 pad 1: Net-(J4-Pin_1) -> VCC
- J4 pad 2: /LED_Output_ch1 -> Net-(J4-Pin_2)
- J6 pad 1: Net-(J4-Pin_1) -> VCC
- J6 pad 2: /LED_Output_ch2 -> Net-(J6-Pin_2)
- J7 pad 1: /LED_Input_ch1 -> /LED_Input_ch2
- J7 pad 2: /LED_Input_ch2 -> /LED_Input_ch1
- J8 pad 1: +5V -> VCC
- U3 pad 1: /LED_Input_ch1 -> /LED_Input_ch2
- U3 pad 3: /LED_Input_ch2 -> /LED_Input_ch1
- U3 pad 4: /LED_Output_ch2 -> /LED_Output_ch1
- U3 pad 6: /LED_Output_ch1 -> /LED_Output_ch2
Routing:
- net VCC: track 97.7 -> 180.9 mm, vias 0 -> 2
- net Net-(J4-Pin_1): track 49.5 -> 0.00 mm
- net Net-(J6-Pin_2): track 0.00 -> 41.9 mm
- net Net-(J4-Pin_2): track 0.00 -> 30.0 mm
- net /LED_Output_ch2: track 23.7 -> 6.96 mm
- net /LED_Output_ch1: track 17.4 -> 4.67 mm
- net /EN: track 0.00 -> 8.94 mm
- net /LED_Input_ch1: track 4.81 -> 9.52 mm
- net /LED_Input_ch2: track 4.54 -> 9.07 mm
- net +5V: track 23.8 -> 26.8 mm
- net GND: vias 6 -> 31
Other:
- board size 49 x 56 mm -> 188.3 x 60.5 mm

Commit message: Fin
Parts:
- removed the H1 at (233.8, 54.5)
- removed the H1 at (300.5, 45.0)
- removed the H1 at (94.5, 59.0)
- removed the H2 at (262.0, 91.0)
- removed the H2 at (56.0, 105.0)
- removed the H2 at (195.3, 100.5)
- removed the H4 at (56.0, 59.0)
- removed the H4 at (262.0, 45.0)
- removed the H4 at (195.3, 54.5)
- removed H5 (x3): MountingHole, MountingHole:MountingHole_4.3mm_M4
- added H1: MountingHole, MountingHole:MountingHole_3.2mm_M3, F.Cu at (156.8, 59.8)
- added H1: MountingHole, MountingHole:MountingHole_3.2mm_M3, F.Cu at (156.8, 105.8)
- added H2: MountingHole, MountingHole:MountingHole_3.2mm_M3, F.Cu at (118.2, 59.8)
- added H4: MountingHole, MountingHole:MountingHole_3.2mm_M3, F.Cu at (118.2, 105.8)
- moved J5 63.8 mm to (119.8, 70.0)
- moved U3 62.8 mm to (125.5, 91.3)
- moved R5 62.8 mm to (131.0, 92.6)
- moved R6 62.8 mm to (133.5, 92.6)
- moved U1 62.3 mm to (129.6, 84.5)
- moved J7 62.3 mm to (118.6, 92.2)
- moved J8 62.3 mm to (118.6, 82.0)
- moved J4 62.1 mm to (127.5, 104.5)
- moved J6 61.7 mm to (141.2, 104.3)
- moved R4 61.6 mm to (123.5, 97.0)
- moved R2 61.5 mm to (126.0, 95.8)
- moved J2 60.6 mm to (130.5, 67.5)
- moved J1 60.6 mm to (134.5, 67.0)
- moved R3 60.0 mm to (133.9, 84.5)
- moved J10 57.2 mm to (151.7, 92.2)
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Routing:
- net VCC: track 180.9 -> 143.5 mm, vias 2 -> 0
- net Net-(J4-Pin_2): track 30.0 -> 21.8 mm
- net Net-(J6-Pin_2): track 41.9 -> 34.7 mm
- net /LED_Input_ch1: track 9.52 -> 6.56 mm
- net /LED_Input_ch2: track 9.07 -> 6.31 mm
- net /EN: track 8.94 -> 6.95 mm
- net /LED_Output_ch1: track 4.67 -> 5.39 mm
- net +5V: track 26.8 -> 26.2 mm
- net GND: vias 31 -> 23
Other:
- board size 188.3 x 60.5 mm -> 40.8 x 52 mm
- board text added: "+"
- board text added: "-"
- board text added: "- PWR input, and daisy chain - 5V LL boost - Aux Breakouts for PWR + Reg"
- board text added: "1"
- board text added: "2"
- board text added: "5V"
- board text added: "CH1"
- board text added: "CH2"
- board text added: "D"
- board text added: "Din"
- board text added: "EN"
- board text added: "For WS2812 (5V supply) or WS2811"
- board text added: "G"
- board text added: "PWR"
- board text added: "UDC LED Driver"

Commit message: Add Prod files
Parts:
- added R1: 1k, Resistor_SMD:R_1206_3216Metric_Pad1.30x1.75mm_HandSolder, F.Cu at (103.0, 59.1)

Commit message: Fin at last
Parts:
- removed R3: 500, Resistor_SMD:R_1206_3216Metric_Pad1.30x1.75mm_HandSolder
- moved R1 39.9 mm to (133.8, 84.5), turned to -90 degrees
Routing:
- net Net-(J4-Pin_2): track 21.8 -> 24.3 mm
- net GND: vias 23 -> 26
